Commit message: Changed trash bin height
Trash bins are now taller, to be more realistic with normal trash bins.
Also, we can use that to make sure the trash doesn't "escape" the trash
bin when being dropped.

File: models/bin.urdf (robot description, URDF)
Before this commit: robot bin, 1 links, 0 joints
Links:
- link bin_body: geometry collision box size=0.01 0.58 0.5; collision box size=0.01 0.58 0.5
