Commit message: Changed conveyor size
In order to support more arms and more trash bins, I changed the size
of the conveyor to a much longer size.

File: models/conveyor/conveyor.urdf (robot description, URDF)
Before this commit: robot myfirst, 1 links, 0 joints
Links:
- link base: geometry collision box size=1 10 0.5; visual box size=1 10 0.5

Commit message: Added per process logging

File: models/conveyor/conveyor.urdf (robot description, URDF)
Before this commit: robot myfirst, 1 links, 0 joints
Links:
- link base: geometry collision box size=1 15 0.5; visual box size=1 15 0.5
