Commit message: Removed texture from trash objects

File: models/YcbCrackerBox/model.urdf (robot description, URDF)
Before this commit: robot model.urdf, 1 links, 0 joints
Links:
- link baseLink: geometry collision mesh filename=collision_vhacd.obj scale=1 1 1

File: models/YcbMasterChefCan/model.urdf (robot description, URDF)
Before this commit: robot model.urdf, 1 links, 0 joints
Links:
- link baseLink: geometry collision mesh filename=collision_vhacd.obj scale=0.7 0.7 0.7

File: models/YcbMustardBottle/model.urdf (robot description, URDF)
Before this commit: robot model.urdf, 1 links, 0 joints
Links:
- link baseLink: geometry collision mesh filename=collision_vhacd.obj scale=1 1 1
