Commit message: Bugfix in UR5 rotational movement

File: assets/ur5/ur5.urdf (robot description, URDF)
Before this commit: robot ur5, 11 links, 10 joints
Joints:
- joint base_link-base_fixed_joint: origin xyz=0 0 0 rpy=0 0 -3.14159265359 -> xyz=0 0 0 rpy=0 0 -31.4159265359
- joint elbow_joint: limit lower=-3.14159265359 upper=3.14159265359 effort=150.0 velocity=3.15 -> lower=-31.4159265359 upper=31.4159265359 effort=150.0 velocity=3.15
- joint shoulder_lift_joint: limit lower=-6.28318530718 upper=6.28318530718 effort=150.0 velocity=3.15 -> lower=-62.8318530718 upper=62.8318530718 effort=150.0 velocity=3.15
- joint shoulder_pan_joint: limit lower=-6.28318530718 upper=6.28318530718 effort=150.0 velocity=3.15 -> lower=-62.8318530718 upper=62.8318530718 effort=150.0 velocity=3.15
- joint wrist_1_joint: limit lower=-6.28318530718 upper=6.28318530718 effort=28.0 velocity=3.2 -> lower=-62.8318530718 upper=62.8318530718 effort=28.0 velocity=3.2
- joint wrist_2_joint: limit lower=-6.28318530718 upper=6.28318530718 effort=28.0 velocity=3.2 -> lower=-62.8318530718 upper=62.8318530718 effort=28.0 velocity=3.2
- joint wrist_3_joint: limit lower=-6.28318530718 upper=6.28318530718 effort=28.0 velocity=3.2 -> lower=-62.8318530718 upper=62.8318530718 effort=28.0 velocity=3.2
